Commit message: Фикс полного запуска: модель, поворот (skid-steer), Nav2, сенсоры
Первый полный запуск системы (Gazebo + Nav2 + SLAM + FSM) выявил
ряд блокирующих багов. Исправлено:

- agv_sensor_processing: добавлен флаг +x скриптам sensor_fusion.py и
  lidar_processing.py — без него ROS не видел их как исполняемые узлы
  при --symlink-install, и запуск сенсоров падал.
- nav2_params.yaml: плагин BackUp переименован back_up -> backup (иначе
  bt_navigator не находит action-сервер и весь стек Nav2 не активируется);
  z_voxels уменьшен 20 -> 16 (максимум для VoxelLayer).
- tractor.urdf.xacro: лидар поднят выше GPS-антенны (z 0.39 -> 0.6,
  ~1.8м над землёй) — раньше GPS попадал в плоскость 2D-сканирования и
  создавал кольцо фантомных препятствий ~0.4м.
- tractor.urdf.xacro: ось колёс 0 0 1 -> 0 0 -1 — команда «вперёд»
  гнала трактор назад, из-за чего Nav2 уводил робота от цели.
- tractor.gazebo.xacro: настройка skid-steer поворота. Передние
  (пассивные) колёса mu=0.0 (скользят вбок), задние mu1=1.0/mu2=0.5,
  max_wheel_torque 500 -> 5000, max_wheel_acceleration 5 -> 15. Раньше
  высокое трение всех 4 колёс стопорило разворот.
- decision_node.py: порог отсечки самозасветки лидара 0.4 -> 0.5 —
  убирает мелькание AVOIDING_OBSTACLE на границе min_range лидара.
- agv_bringup/CMakeLists.txt: установка config/ только если папка есть.

После правок трактор едет прямо, разворачивается и доходит до точек
маршрута покрытия; runaway устранён.

Co-Authored-By: Claude Opus 4.8 <noreply@anthropic.com>

File: src/agv_description/urdf/tractor.urdf.xacro (robot description, xacro)
@@ -83,5 +83,8 @@
       <origin xyz="${x_pos} ${y_pos} ${-ground_clearance + wheel_radius - chassis_height/2}"
               rpy="${pi/2} 0 0"/>
-      <axis xyz="0 0 1"/>
+      <!-- Ось -Z: при rpy=pi/2 вокруг X положительное вращение даёт движение
+           ВПЕРЁД (+X). С осью +Z трактор ехал назад на команду «вперёд»,
+           что ломало навигацию (Nav2 уводил робота от цели). -->
+      <axis xyz="0 0 -1"/>
       <!-- Трение и демпфирование для стабильной физики -->
       <dynamics damping="0.1" friction="1.0"/>
@@ -246,6 +249,10 @@
     <parent link="cabin_link"/>
     <child  link="lidar_link"/>
-    <!-- Спереди кабины, на крыше — хороший обзор вперёд -->
-    <origin xyz="0.35 0 0.39" rpy="0 0 0"/>
+    <!-- Спереди кабины, на мачте выше GPS-антенны.
+         Важно: плоскость 2D-сканирования должна идти ВЫШЕ всех конструкций
+         трактора (кабина, GPS), иначе лидар «видит» сам трактор как кольцо
+         фантомных препятствий на ~0.4м и блокирует навигацию.
+         z=0.6 (система кабины) ≈ 1.8м над землёй, выше верха GPS (1.63м). -->
+    <origin xyz="0.35 0 0.6" rpy="0 0 0"/>
   </joint>
   <!-- == RGB Камера (спереди корпуса, ориентирована вперёд) == -->

File: src/agv_gazebo/urdf/tractor.gazebo.xacro (robot description, xacro)
@@ -21,8 +21,13 @@
     <material>Gazebo/DarkGreen</material>
   </gazebo>
+  <!-- Передние колёса — пассивные, с НИЗКИМ трением.
+       Трактор поворачивает по принципу skid-steer (разворот за счёт разной
+       скорости задних колёс). При высоком трении всех 4 колёс боковое
+       сопротивление не даёт развернуться — привод стопорится. Низкое трение
+       передних колёс позволяет им скользить вбок, и трактор может поворачивать. -->
   <gazebo reference="front_left_wheel_link">
     <material>Gazebo/DarkGrey</material>
-    <mu1>1.0</mu1>
-    <mu2>1.0</mu2>
+    <mu1>0.0</mu1>
+    <mu2>0.0</mu2>
     <kp>1e6</kp>
     <kd>100.0</kd>
@@ -30,13 +35,15 @@
   <gazebo reference="front_right_wheel_link">
     <material>Gazebo/DarkGrey</material>
-    <mu1>1.0</mu1>
-    <mu2>1.0</mu2>
+    <mu1>0.0</mu1>
+    <mu2>0.0</mu2>
     <kp>1e6</kp>
     <kd>100.0</kd>
   </gazebo>
+  <!-- Задние (ведущие) колёса — сцепление для тяги (mu1), но умеренное
+       боковое трение (mu2), чтобы они тоже могли подскальзывать при развороте. -->
   <gazebo reference="rear_left_wheel_link">
     <material>Gazebo/DarkGrey</material>
-    <mu1>1.5</mu1>
-    <mu2>1.5</mu2>
+    <mu1>1.0</mu1>
+    <mu2>0.5</mu2>
     <kp>1e6</kp>
     <kd>100.0</kd>
@@ -44,6 +51,6 @@
   <gazebo reference="rear_right_wheel_link">
     <material>Gazebo/DarkGrey</material>
-    <mu1>1.5</mu1>
-    <mu2>1.5</mu2>
+    <mu1>1.0</mu1>
+    <mu2>0.5</mu2>
     <kp>1e6</kp>
     <kd>100.0</kd>
@@ -68,6 +75,8 @@
       <!-- Диаметр = 2 * wheel_radius = 0.6 м -->
       <wheel_diameter>0.6</wheel_diameter>
-      <max_wheel_torque>500.0</max_wheel_torque>
-      <max_wheel_acceleration>5.0</max_wheel_acceleration>
+      <!-- Момент повышен до 1500: при развороте нужно преодолеть боковое
+           трение колёс. max_wheel_acceleration повышено для отзывчивости. -->
+      <max_wheel_torque>5000.0</max_wheel_torque>
+      <max_wheel_acceleration>15.0</max_wheel_acceleration>
       <!-- Публиковать одометрию в топик /odom — ДА (её читает локальный EKF).
            Публиковать TF odom->base_link — НЕТ: иначе конфликт с локальным EKF,
